File: ECAD/Custom_Calculator.kicad_sch (KiCad schematic)
At the start: 98 parts, among them SW1 SW_SPST, SW10 SW_SPST, SW11 SW_SPST, SW12 SW_SPST, SW13 SW_SPST, SW14 SW_SPST, SW15 SW_SPST, SW16 SW_SPST, SW17 SW_SPST, SW18 SW_SPST, SW19 SW_SPST, SW2 SW_SPST, SW20 SW_SPST, SW21 SW_SPST, SW22 SW_SPST, SW23 SW_SPST, SW24 SW_SPST, SW25 SW_SPST, SW26 SW_SPST, SW27 SW_SPST, SW28 SW_SPST, SW29 SW_SPST, SW3 SW_SPST, SW30 SW_SPST, SW31 SW_SPST, SW32 SW_SPST, SW33 SW_SPST, SW34 SW_SPST, SW35 SW_SPST, SW36 SW_SPST, SW37 SW_SPST, SW38 SW_SPST, SW39 SW_SPST, SW4 SW_SPST, SW40 SW_SPST, SW41 SW_SPST, SW42 SW_SPST, SW43 SW_SPST, SW44 SW_SPST, SW45 SW_SPST, SW46 SW_SPST, SW47 SW_SPST, SW48 SW_SPST, SW49 SW_SPST, SW5 SW_SPST, SW50 SW_SPST, SW51 SW_SPST, SW52 SW_SPST, SW53 SW_SPST, SW54 SW_SPST, SW55 SW_SPST, SW56 SW_SPST, SW57 SW_SPST, SW58 SW_SPST, SW59 SW_SPST, SW6 SW_SPST, SW60 SW_SPST, SW61 SW_SPST, SW62 SW_SPST, SW63 SW_SPST, SW64 SW_SPST, SW65 SW_SPST, SW66 SW_SPST, SW67 SW_SPST, SW68 SW_SPST, SW69 SW_SPST, SW7 SW_SPST, SW70 SW_SPST, SW71 SW_SPST, SW72 SW_SPST, SW73 SW_SPST, SW74 SW_SPST, SW75 SW_SPST, SW76 SW_SPST, SW77 SW_SPST, SW78 SW_SPST, SW79 SW_SPST, SW8 SW_SPST, SW80 SW_SPST, SW81 SW_SPST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

Commit message: Added connections to  MCP23017 and added notation to rows
Connections:
- net ROW 1: now also SW1.1 (A), SW13.1 (A), SW19.1 (A), SW25.1 (A), SW31.1 (A), SW37.1 (A), SW43.1 (A), SW49.1 (A), SW55.1 (A), SW61.1 (A), SW67.1 (A), SW7.1 (A), SW73.1 (A), SW79.1 (A), SW85.1 (A), SW91.1 (A)
- net ROW 2: now also SW14.1 (A), SW2.1 (A), SW20.1 (A), SW26.1 (A), SW32.1 (A), SW38.1 (A), SW44.1 (A), SW50.1 (A), SW56.1 (A), SW62.1 (A), SW68.1 (A), SW74.1 (A), SW8.1 (A), SW80.1 (A), SW86.1 (A), SW92.1 (A)
- net ROW 3: now also SW15.1 (A), SW21.1 (A), SW27.1 (A), SW3.1 (A), SW33.1 (A), SW39.1 (A), SW45.1 (A), SW51.1 (A), SW57.1 (A), SW63.1 (A), SW69.1 (A), SW75.1 (A), SW81.1 (A), SW87.1 (A), SW9.1 (A), SW93.1 (A)
- net ROW 4: now also SW10.1 (A), SW16.1 (A), SW22.1 (A), SW28.1 (A), SW34.1 (A), SW4.1 (A), SW40.1 (A), SW46.1 (A), SW52.1 (A), SW58.1 (A), SW64.1 (A), SW70.1 (A), SW76.1 (A), SW82.1 (A), SW88.1 (A), SW94.1 (A)
- net ROW 5: now also SW11.1 (A), SW17.1 (A), SW23.1 (A), SW29.1 (A), SW35.1 (A), SW41.1 (A), SW47.1 (A), SW5.1 (A), SW53.1 (A), SW59.1 (A), SW65.1 (A), SW71.1 (A), SW77.1 (A), SW83.1 (A), SW89.1 (A)
- net ROW 6: now also SW12.1 (A), SW18.1 (A), SW24.1 (A), SW30.1 (A), SW36.1 (A), SW42.1 (A), SW48.1 (A), SW54.1 (A), SW6.1 (A), SW60.1 (A), SW66.1 (A), SW72.1 (A), SW78.1 (A), SW84.1 (A), SW90.1 (A)

Commit message: Completed Schematic and changed spreadsheet specs
Parts:
- added C1: 0.1 uF, symbol Device:C
Connections:
- net +3V3: now also U2.18 (~{RESET}), U2.9 (V_{DD}), C1.1
- net GND: now also U2.10 (V_{SS}), U2.15 (A0), U2.16 (A1), U2.17 (A2), C1.2
- net COL #9: now reaches U2.1 (GPB0)
- net at U2.12 (SCK): now also U1.26 (19_A5_SCL0)
- net at U2.13 (SDA): now also U1.25 (18_A4_SDA0)
- net COL #10: now reaches U2.2 (GPB1)
- net at U2.20 (INTA): now also U1.27 (20_A6_TX5_LRCLK1)
- net COL #1: now reaches U2.21 (GPA0)
- net COL #2: now reaches U2.22 (GPA1)
- net COL #3: now reaches U2.23 (GPA2)
- net COL #4: now reaches U2.24 (GPA3)
- net COL #5: now reaches U2.25 (GPA4)
- net COL #6: now reaches U2.26 (GPA5)
- net COL #7: now reaches U2.27 (GPA6)
- net COL #8: now reaches U2.28 (GPA7)
- net COL #11: now reaches U2.3 (GPB2)
- net COL #12: now reaches U2.4 (GPB3)
- net COL #13: now reaches U2.5 (GPB4)
- net COL #14: now reaches U2.6 (GPB5)
- net COL #15: now reaches U2.7 (GPB6)
- net COL #16: now reaches U2.8 (GPB7)
- no-connect marks 1 -> 36
